File: doc/cad/doorbell/doorbell.kicad_pcb (KiCad board)
At the start: 2 copper layers, 23 parts, among them J1 Doorbell PCB, J2 12V Supply, J3 Speaker, T1 Transformer_1P_1S, U1 ESP32-WROOM-32, U2 TDA1517P/N3_112, U3 AMS1117-3.3

Commit message: updated pcb
Parts:
- added REF**: MountingHole_3mm_Pad, MountingHole:MountingHole_3mm_Pad, F.Cu at (211.5, 42.5)
- added REF**: MountingHole_3mm_Pad, MountingHole:MountingHole_3mm_Pad, F.Cu at (84.5, 42.5)
- added REF**: MountingHole_3mm_Pad, MountingHole:MountingHole_3mm_Pad, F.Cu at (85.0, 150.5)
- added REF**: MountingHole_3mm_Pad, MountingHole:MountingHole_3mm_Pad, F.Cu at (211.0, 150.5)
- moved C6 24.9 mm to (207.2, 111.0)
- moved C9 20.1 mm to (199.5, 131.0), turned to 180 degrees
- moved J3 15.9 mm to (211.0, 130.0)
- moved R1 14.3 mm to (141.4, 48.7)
- moved C11 14.3 mm to (99.2, 70.7)
- moved R3 14.3 mm to (99.2, 88.8)
- moved U1 14.3 mm to (116.0, 54.1)
- moved C8 6.42 mm to (199.5, 142.8), turned to 180 degrees
- moved C10 3.77 mm to (182.0, 140.8), turned to 90 degrees
- moved C7 3.64 mm to (183.0, 107.5), turned to -90 degrees
- moved C4 2.50 mm to (184.0, 100.0)
- moved C5 2.07 mm to (184.0, 120.0)
Connections:
- net Net-(J1-Pin_1) renamed +3.3V
Routing:
- net +12V: track 27.9 -> 154.4 mm
- net +3.3V: track 43.9 -> 150.5 mm, vias 0 -> 2
- net Net-(U2-OUT1): track 0.00 -> 43.6 mm
- net Net-(U2-SVRR): track 0.00 -> 17.4 mm
- net GND: track 39.8 -> 24.3 mm, vias 0 -> 4
- net Net-(J1-Pin_3): track 91.6 -> 77.3 mm
- net Net-(U2--INV2): track 0.00 -> 11.7 mm
- net Net-(U2--INV1): track 9.52 -> 16.9 mm

Commit message: verified initial pcb
Parts:
- added REF**: , MountingHole:MountingHole_2.5mm_Pad, F.Cu at (109.0, 115.5)
- added REF**: MountingHole_2.5mm_Pad, MountingHole:MountingHole_2.5mm_Pad, F.Cu at (109.0, 97.5)
- J1 Doorbell PCB: renamed from J1
- J2 +12VDC: renamed from J2
- J3 Speaker: renamed from J3
- moved J3 Speaker 42.5 mm to (211.0, 87.5)
- moved C10 28.1 mm to (163.4, 119.7)
- moved C4 28.1 mm to (165.4, 79.0)
- moved C5 28.1 mm to (165.4, 99.0)
- moved C7 28.1 mm to (164.4, 86.5)
- moved C8 28.1 mm to (180.9, 121.7)
- moved C9 28.1 mm to (180.9, 110.0)
- moved U2 28.1 mm to (174.9, 80.4)
- moved R2 28.1 mm to (159.3, 73.5)
- moved R3 24.9 mm to (116.1, 70.5), turned to 180 degrees
- moved REF** 22.8 mm to (95.0, 130.0)
- moved REF** 20.5 mm to (211.0, 130.0)
- moved REF** 15.9 mm to (95.0, 54.5)
- moved C6 15.5 mm to (192.5, 106.0)
- moved C11 10.7 mm to (108.5, 76.0), turned to 0 degrees
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Routing:
- net +12V: track 154.4 -> 125.7 mm
- net Net-(R2-Pad2): track 8.92 -> 37.3 mm
- net Net-(J3-Pin_1): track 0.00 -> 24.6 mm
- net +3.3V: track 150.5 -> 125.9 mm
- net Net-(U2-OUT1): track 43.6 -> 31.5 mm
- net Net-(U1-EN): track 34.5 -> 30.4 mm
- added copper zone on B.Cu, net GND
- added copper zone on F.Cu, net GND
Other:
- board outline added: 128.5 x 99 mm
- board text added: "Doorbell PCB"

Commit message: Minor improvements
Parts:
- J3 SPK: renamed from J3 Speaker
- RV1 VOL: renamed from RV1; footprint Potentiometer_THT:Potentiometer_Piher_PT-10-V10_Vertical_Hole -> Potentiometer_THT:Potentiometer_Piher_PT-15-H05_Horizontal
- moved RV1 VOL 20.0 mm to (211.5, 95.0), turned to 180 degrees
- moved J3 SPK 17.5 mm to (210.5, 105.0)
- moved REF** 8.00 mm to (95.0, 122.0)
- moved REF** 8.00 mm to (211.0, 122.0)
- moved REF** 6.96 mm to (111.5, 109.0)
- moved REF** 6.96 mm to (111.5, 91.0)
- moved C12 4.00 mm to (173.5, 58.0)
- moved C2 4.00 mm to (165.5, 59.5)
- moved C1 3.50 mm to (148.5, 56.5)
Routing:
- net Net-(T1-SB): track 15.3 -> 38.1 mm
- net Net-(R2-Pad2): track 37.3 -> 49.2 mm
- net Net-(J3-Pin_1): track 24.6 -> 14.6 mm
- net +3.3V: track 125.9 -> 119.9 mm
- net GND: track 24.3 -> 18.8 mm
Other:
- board size 128.5 x 99 mm -> 128.5 x 91.5 mm

Commit message: Added testing hackRF rf captures. Schematic updates.
Parts:
- added G***: LOGO, images:creationfactory, F.Cu at (106.5, 122.5)
- J1: renamed from J1 Doorbell PCB
- J2: renamed from J2 +12VDC
- J3: renamed from J3 SPK
- RV1: renamed from RV1 VOL
Connections:
- J1 pad 6: unconnected-(J1-Pin_6-Pad6) -> Net-(J1-Pin_6)
- J1 pad 7: unconnected-(J1-Pin_7-Pad7) -> Net-(J1-Pin_7)
- T1 pad 1: Net-(J1-Pin_5) -> Net-(J1-Pin_7)
- T1 pad 2: Net-(J1-Pin_4) -> Net-(J1-Pin_6)
- U1 pad 28: unconnected-(U1-IO17-Pad28) -> Net-(J1-Pin_5)
- U1 pad 30: unconnected-(U1-IO18-Pad30) -> Net-(J1-Pin_4)
Routing:
- net Net-(J1-Pin_5): track 19.7 -> 81.1 mm, vias 0 -> 1
- net Net-(J1-Pin_4): track 19.7 -> 77.6 mm, vias 0 -> 1
- net Net-(J1-Pin_6): track 0.00 -> 21.3 mm
- net Net-(J1-Pin_7): track 0.00 -> 18.0 mm
- net +3.3V: track 119.9 -> 124.1 mm, vias 2 -> 3
- net GND: vias 4 -> 34
Other:
- board text added: "Luis Teixeira 2026 https://creationfactory.co"
