File: doc/cad/doorbell/doorbell.kicad_pcb (KiCad board)
At the start: 2 copper layers, 128.5 x 91.5 mm, 32 parts, among them J1 Bell PCB Conn, J2 +12VDC, J3 Speaker, J4 UART, T1 Transformer_1P_1S, U1 ESP32-WROOM-32, U2 TDA1517P/N3_112, U3 AMS1117-3.3

Commit message: Improvements
Routing:
- net GND: track 18.8 -> 8.57 mm
- net +3.3V: track 165.2 -> 171.5 mm
Other:
- board text added: "+"
- board text added: "12VDC"
- board text removed: "+12VDC"
Changed lines of the file:
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@@
 		(fill no)
 		(layer "F.Cu")
-		(net "/TX")
 	)
 	(gr_rect
@@
 		)
 	)
-	(gr_text "+12VDC"
-		(at 153.261689 46.699526 0)
+	(gr_text "+"
+		(at 152 42.5 0)
+		(layer "F.SilkS")
+		(effects
+			(font
+				(size 1 1)
+				(thickness 0.25)
+				(bold yes)
+			)
+			(justify left bottom)
+		)
+	)
+	(gr_text "12VDC"
+		(at 154 46.699526 0)
 		(layer "F.SilkS")
 		(effects
@@
 		)
 	)
+	(gr_text "+"
+		(at 211 102.5 90)
+		(layer "F.SilkS")
+		(effects
+			(font
+				(size 1 1)
+				(thickness 0.25)
+				(bold yes)
+			)
+			(justify left bottom)
+		)
+	)
 	(gr_text "SPK"
 		(at 214 107 90)
@@
 	)
 	(segment
+		(start 168.5 63.35)
+		(end 167.15 62)
+		(width 0.8)
+		(layer "F.Cu")
+		(net "+3.3V")
+	)
+	(segment
 		(start 177.35 57.85)
 		(end 181.35 57.85)
@@
 	)
 	(segment
+		(start 160.85 62)
+		(end 167.15 62)
+		(width 1.5)
+		(layer "F.Cu")
+		(net "+3.3V")
+	)
+	(segment
 		(start 173.35 59.35)
 		(end 175.85 59.35)
@@
 	)
 	(segment
+		(start 169.35 63.35)
+		(end 168.5 63.35)
+		(width 0.8)
+		(layer "F.Cu")
+		(net "+3.3V")
+	)
+	(segment
 		(start 107.25 47.135)
 		(end 112.635 47.135)
@@
 	)
 	(segment
-		(start 168.5 63.35)
-		(end 167.15 62)
-		(width 0.8)
-		(layer "F.Cu")
-		(net "+3.3V")
-	)
-	(segment
 		(start 127.17 67.17)
 		(end 126.84 67.5)
@@
 		(net "+3.3V")
 	)
-	(segment
-		(start 169.35 63.35)
-		(end 168.5 63.35)
-		(width 0.8)
-		(layer "F.Cu")
-		(net "+3.3V")
-	)
 	(via
 		(at 169.35 63.35)
@@
 	)
 	(segment
-		(start 199.5 73)
-		(end 202.5 70)
-		(width 0.2)
-		(layer "F.Cu")
-		(net "GND")
-	)
-	(segment
 		(start 163.88 114.24)
 		(end 163.38 114.74)
-		(width 0.2)
-		(layer "F.Cu")
-		(net "GND")
-	)
-	(segment
-		(start 199.5 79)
-		(end 199.5 73)
 		(width 0.2)
 		(layer "F.Cu")
@@
 		)
 		(min_thickness 0.25)
-		(fill yes
+		(fill
 			(thermal_gap 0.5)
 			(thermal_bridge_width 0.5)
@@
 		(polygon
 			(pts
-				(xy 148 38.1035) (xy 148 44.5) (xy 105.5 44.5) (xy 90 56.5) (xy 90 78) (xy 147 78) (xy 147 126.5)
+				(xy 152 38.0989) (xy 148 42) (xy 148 44.5) (xy 105.5 44.5) (xy 90 56.5) (xy 90 78) (xy 147 78) (xy 147 126.5)
 				(xy 215.5 126.5) (xy 215.5 38)
 			)
@@
 		)
 		(min_thickness 0.25)
-		(fill yes
+		(fill
 			(thermal_gap 0.5)
 			(thermal_bridge_width 0.5)
@@
 		(polygon
 			(pts
-				(xy 148 38.1035) (xy 148 44.5) (xy 105.5 44.5) (xy 90 56.5) (xy 90 78) (xy 147 78) (xy 147 126.5)
-				(xy 215.5 126.5) (xy 215.5 38)
-			)
-		)
+				(xy 152 38.100433) (xy 148 42) (xy 148 44.5) (xy 105.5 44.5) (xy 90 56.5) (xy 90 78) (xy 147 78)
+				(xy 147 126.5) (xy 215.5 126.5) (xy 215.5 38)
+			)
+		)

Commit message: pcb annotations
Other:
- board text added: "Kinetic Doorbell Wifi Expansion REV 1.0 2026-09 Luis Teixeira https://creationfactory.co"
- board text removed: "Luis Teixeira 2026 https://creationfactory.co"
Changed lines of the file:
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@@
 		(layer "Edge.Cuts")
 	)
-	(gr_text "Luis Teixeira 2026\nhttps://creationfactory.co"
+	(gr_text "Kinetic Doorbell Wifi Expansion\nREV 1.0 2026-09\nLuis Teixeira https://creationfactory.co"
 		(at 113.5 125.5 0)
 		(layer "F.SilkS")
@@
 		)
 		(min_thickness 0.25)
-		(fill
+		(fill yes
 			(thermal_gap 0.5)
 			(thermal_bridge_width 0.5)
@@
 		)
 		(min_thickness 0.25)
-		(fill
+		(fill yes
 			(thermal_gap 0.5)
 			(thermal_bridge_width 0.5)
